File: trap-pcb/_saved_trap-pcb.sch (KiCad schematic (older format))
At the start: 41 parts, among them J1 PIR_1, J2 PIR_2, J3 PIR_3, J4 Power In, K1 RELAY, K2 RELAY, M1 Motor_Servo_1, M2 Motor_Servo_2, M3 Motor_DC, P1 Digital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

Commit message: updated pcb
Parts:
- removed R1, R2, R7, R8: 100k, Resistors_SMD:R_1206_HandSoldering, symbol Device:R
- added C5: 6800uF, Capacitors_THT:CP_Radial_D18.0mm_P7.50mm, symbol device:C
- added D3: D, Diodes_THT:D_A-405_P7.62mm_Horizontal, symbol Device:D
- added K3: RELAY, Relays_THT:Relay_SPDT_SANYOU_SRD_Series_Form_C, symbol SeeedOPL-Relay-2016:RELAY-HLS8L-DC3V-S-C_5P-19X15MM_
- added MK1, MK2, MK3, MK4: Mounting_Hole, Mounting_Holes:MountingHole_4.3mm_M4_Pad_Via, symbol Mechanical:Mounting_Hole
- D1, D2: footprint Diodes_SMD:D_SOD-323_HandSoldering -> Diodes_THT:D_A-405_P7.62mm_Horizontal; Digikey 1N4148XTPMSCT-ND -> 1N4007-TPMSCT-ND
- Q1: footprint TO_SOT_Packages_SMD:SOT-223-3Lead_TabPin2 -> TO_SOT_Packages_SMD:SOT-23; Digikey NTF3055L108T1GOSCT-ND -> 785-1015-1-ND
Connections:
- net labels removed: A0, A1, A2, A3, A4, A5
- wire segments 196 -> 188
- no-connect marks 8 -> 17
Other:
- moved on the sheet: C1, C2, C3, C4, D1, D2, K1, K2, L1, M1, M2, M3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
