File: trap-pcb/trap-pcb.kicad_pcb (KiCad board)
At the start: 2 copper layers, 114 x 120 mm, 45 parts, among them J1 PIR_1, J2 PIR_2, J3 PIR_3, J4 Power In, K1 RELAY, K2 RELAY, M1 Motor_Servo_1, M2 Motor_Servo_2, M3 Motor_DC, P1 Digital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

Commit message: updated pcb
Parts:
- removed R1, R2, R7, R8: 100k, Resistors_SMD:R_1206_HandSoldering
- removed REF** (x4): MountingHole_4.3mm_M4_Pad_Via, Mounting_Holes:MountingHole_4.3mm_M4_Pad_Via
- added C5: 6800uF, Capacitors_THT:CP_Radial_D18.0mm_P7.50mm, F.Cu at (132.2, 58.2)
- added D3: D, Diodes_THT:D_A-405_P7.62mm_Horizontal, F.Cu at (185.0, 134.0)
- added K3: RELAY, Relays_THT:Relay_SPDT_SANYOU_SRD_Series_Form_C, F.Cu at (189.2, 138.0)
- added MK1: Mounting_Hole, Mounting_Holes:MountingHole_4.3mm_M4_Pad_Via, F.Cu at (175.0, 40.0)
- added MK2: Mounting_Hole, Mounting_Holes:MountingHole_4.3mm_M4_Pad_Via, F.Cu at (125.2, 40.0)
- added MK3: Mounting_Hole, Mounting_Holes:MountingHole_4.3mm_M4_Pad_Via, F.Cu at (175.0, 150.0)
- added MK4: Mounting_Hole, Mounting_Holes:MountingHole_4.3mm_M4_Pad_Via, F.Cu at (125.0, 150.0)
- D1, D2: footprint Diodes_SMD:D_SOD-323_HandSoldering -> Diodes_THT:D_A-405_P7.62mm_Horizontal
- Q1: footprint TO_SOT_Packages_SMD:SOT-223-3Lead_TabPin2 -> TO_SOT_Packages_SMD:SOT-23
- SW3: value Retracted -> Extended
- SW4: value Extended -> Retracted
- moved D2 36.3 mm to (210.6, 104.0), turned to 180 degrees
- moved C1 35.6 mm to (199.8, 93.7)
- moved M3 35.6 mm to (208.3, 93.9)
- moved Q2 30.8 mm to (194.6, 76.9)
- moved R4 30.8 mm to (190.5, 77.2)
- moved M1 30.8 mm to (208.5, 81.7)
- moved M2 30.8 mm to (208.5, 63.7)
- moved K1 30.3 mm to (204.0, 109.2), turned to 270 degrees
- moved R5 29.4 mm to (189.8, 59.4)
- moved Q3 29.4 mm to (194.7, 58.6)
- moved Q4 25.4 mm to (195.0, 99.7), turned to 90 degrees
- moved Q1 22.9 mm to (178.0, 138.6), turned to 0 degrees
- moved C3 18.8 mm to (157.6, 55.6)
- moved C4 18.8 mm to (177.1, 52.8)
- moved L1 18.8 mm to (152.3, 56.1)
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Connections:
- P1 pad 10: /Motor_forward -> Net-(P1-Pad10)
- P1 pad 11: /Motor_back -> Net-(P1-Pad11)
- P2 pad 1: +5V -> Net-(P2-Pad1)
- P2 pad 10: /A2 -> /Motor_back
- P2 pad 11: /A1 -> /Retracted
- P2 pad 12: /A0 -> /Extended
- P2 pad 4: Net-(P2-Pad4) -> +5V
- P2 pad 5: /Extended -> Net-(P2-Pad5)
- P2 pad 6: /Retracted -> Net-(P2-Pad6)
- P2 pad 7: /A5 -> /Servo_1_power
- P2 pad 8: /A4 -> /Servo_2_power
- P2 pad 9: /A3 -> /Motor_forward
- P7 pad 10: /Motor_forward -> Net-(P7-Pad10)
- P7 pad 11: /Motor_back -> Net-(P7-Pad11)
- P8 pad 1: +5V -> Net-(P8-Pad1)
- P8 pad 10: /A2 -> /Motor_back
- P8 pad 11: /A1 -> /Retracted
- P8 pad 12: /A0 -> /Extended
- P8 pad 4: Net-(P8-Pad4) -> +5V
- P8 pad 5: /Extended -> Net-(P8-Pad5)
- P8 pad 6: /Retracted -> Net-(P8-Pad6)
- P8 pad 7: /A5 -> /Servo_1_power
- P8 pad 8: /A4 -> /Servo_2_power
- P8 pad 9: /A3 -> /Motor_forward
- Q1 pad 3: Net-(K1-Pad5) -> Net-(D3-Pad2)
- SW1 pad 2: +5V -> GND
Routing:
- net +5V: track 312.7 -> 241.3 mm
- net /Servo_1_power: track 2.38 -> 58.4 mm
- net /Servo_2_power: track 3.78 -> 45.4 mm
- net /Retracted: track 103.1 -> 77.9 mm, vias 2 -> 1
- net /Motor_back: track 46.6 -> 71.5 mm
- net VCC: track 259.3 -> 236.5 mm
- net Net-(D1-Pad2): track 36.3 -> 59.0 mm
- net /Motor_forward: track 41.7 -> 64.2 mm
- net /Extended: track 94.0 -> 71.5 mm, vias 2 -> 1
- net Net-(D3-Pad2): track 0.00 -> 21.6 mm
- net Net-(K1-Pad5): track 12.5 -> 28.8 mm
- net GND: track 51.5 -> 35.2 mm, vias 16 -> 7
- net /H_bridge_back: track 86.8 -> 75.6 mm
- net /A5: track 7.67 -> 0.00 mm
- net /A3: track 7.67 -> 0.00 mm
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- added copper zone on F.Cu, net +5V
- removed copper zone on F.Cu, net GND
Other:
- board text added: "+12V"
- board text removed: "+24V"
