File: trap-pcb/trap-pcb.sch (KiCad schematic (older format))
At the start: 41 parts, among them J1 PIR_1, J2 PIR_2, J3 PIR_3, J4 Power In, K1 RELAY, K2 RELAY, M1 Motor_Servo_1, M2 Motor_Servo_2, M3 Motor_DC, P1 Digital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

Commit message: updated pcb
Parts:
- added C5: 6800uF, Capacitors_THT:CP_Radial_D18.0mm_P7.50mm, symbol device:C
- D1, D2: footprint Diodes_SMD:D_SOD-323_HandSoldering -> Diodes_THT:D_A-405_P7.62mm_Horizontal; Digikey 1N4148XTPMSCT-ND -> 1N4007-TPMSCT-ND
- Q1: value Q_NMOS_GSD -> Q_NMOS_GDS; symbol device:Q_NMOS_GSD -> device:Q_NMOS_GDS
- SW3: value Reset -> Extended
- SW4: value Reset -> Retracted
Connections:
- net A4 is gone; now on net Servo_2_power: P2.8 (Pin_8), P8.8 (Pin_8)
- net A5 is gone; now on net Servo_1_power: P2.7 (Pin_7), P8.7 (Pin_7)
- net GND: now also Q1.3 (S), C5.2; no longer Q1.2 (S)
- net VCC: now also C5.1
- net at K1.5 (NC), K2.4 (NO): now also Q1.2 (D); no longer Q1.3 (D)
Other:
- moved on the sheet: C1, C2, C3, C4, D1, D2, K1, K2, L1, M1, M2, M3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
